File: eda/cowboys_vs_dinos/cowboys_vs_dinos.kicad_sch (KiCad schematic)
At the start: 0 parts

Commit message: schematic and poc test work
Parts:
- added BT1: Battery_Lipo, 0_local:Battery_Connector_back, symbol 0_local:Battery_Lipo
- added C10, C11, C12, C20, C21, C22: C_Disc_D3, 0_local:C_Disc_D3_back, symbol 0_local:C_Disc_D3
- added D1, D2, D3, D4, D5, D6, D7, D8, D9: LED_3mm, 0_local:LED_D3.0mm-2-std_back, symbol 0_local:LED_THT_3mm
- added D10, D11, D12, D20, D21, D22: LED_WS2812D_5mm, 0_local:LED_D5.0mm-4_WS2812D_2024_back, symbol 0_local:LED_WS2812D_THT_5mm
- added J1: Battery_Conn, 0_local:Battery_Connector_back, symbol 0_local:Battery_Conn
- added R1, R10, R2, R20, R3, R4, R5, R6, R7, R8, R9: 47R_6.3mm, 0_local:R_Axial_DIN0207_L6.3_D2.5_P7.62_Horiz_back, symbol 0_local:R_Axial_Z_L6.3
- added SW1: SW_SPDT_SS12D00G, 0_local:SW_SPDT_Slide_SS12D00G-1P2T_3pin_back, symbol 0_local:SW_SPDT_SS12D00G
- added TCH1, TCH3, TCH5: SYM_Touch_lg, symbol 0_local:SYM_Touch_lg
- added U1: ESP32-WEMOS-LOLIN32-LITE, 0_local:ESP32_WEMOS_LOLIN32_LITE_back, symbol 0_local:ESP32-WEMOS-LOLIN32-LITE
Connections:
- new net: D20.4 (DIN), R20.1
- new net: D6.1 (K), R6.1
- new net: D1.1 (K), R1.1
- new net: D10.4 (DIN), R10.1
- new net: D9.1 (K), R9.1
- new net: BT1.1 (Pin_1), SW1.2 (B)
- new net: D8.1 (K), R8.1
- new net: D2.1 (K), R2.1
- new net: D3.1 (K), R3.1
- new net: D7.1 (K), R7.1
- new net: D5.1 (K), R5.1
- new net: D4.1 (K), R4.1
- new net +3.3V: C10.1, C11.1, C12.1, C20.1, C21.1, C22.1, D10.2 (VDD), D11.2 (VDD), D12.2 (VDD), D20.2 (VDD), D21.2 (VDD), D22.2 (VDD), U1.3V3 (3v3)
- new net 0: TCH1.1, U1.0 (GPIO0/TCH1)
- new net 12: TCH5.1, U1.12 (GPIO12/TCH5)
- new net 14: D1.2 (A), U1.14 (GPIO14/TCH6)
- new net 15: TCH3.1, U1.15 (GPIO15/TCH3)
- new net 16: R20.2, U1.16 (GPIO16)
- new net 17: R10.2, U1.17 (GPIO17)
- new net 18: D8.2 (A), U1.18 (GPIO18)
- new net 23: D9.2 (A), U1.23 (GPIO23)
- new net 25: D4.2 (A), U1.25 (GPIO25)
- new net 26: D3.2 (A), U1.26 (GPIO26)
- new net 27: D2.2 (A), U1.27 (GPIO27/TCH7)
- new net 32: D6.2 (A), U1.32 (GPIO32/TCH9)
- new net 33: D5.2 (A), U1.33 (GPIO33/TCH8)
- new net 5: D7.2 (A), U1.5 (GPIO5)
- new net D10: D10.1 (DOUT), D11.4 (DIN)
- new net D11: D11.1 (DOUT), D12.4 (DIN)
- new net D20: D20.1 (DOUT), D21.4 (DIN)
- new net D21: D21.1 (DOUT), D22.4 (DIN)
- new net GBAT: BT1.2 (Pin_2), J1.2 (Pin_2)
- new net GND: C10.2, C11.2, C12.2, C20.2, C21.2, C22.2, D10.3 (GND), D11.3 (GND), D12.3 (GND), D20.3 (GND), D21.3 (GND), D22.3 (GND), R1.2, R2.2, R3.2, R4.2, R5.2, R6.2, R7.2, R8.2, R9.2, U1.GND
- new net VBAT: J1.1 (Pin_1), SW1.1 (A)
- no-connect marks 0 -> 13
Other:
- note added: "Addressable LEDs"
- note added: "Capacitive Touch"
- note added: "Power"
- note added: "Traditional 2-Pin LEDs"
- note added: "VBAT & GBAT + -"
- note added: "WARNING: JST-PH connector wired reverse polarity from many cables Black wire might go to + & red to - It depends on cable pinout so... DOUBLE CHECK BEFORE CONNECTING!"
- note added: "|- Input ONLY -|"
- company: (none) -> Crafted by @alt_bier a.k.a. Richard Gowen and his Badge Team
- title: (none) -> Cowboys_vs_Dinos

Commit message: center art
Parts:
- added TCH3, TCH5: SYM_Touch_lg, symbol 0_local:SYM_Touch_lg
- renumbered TCH3 to TCH2, TCH5 to TCH4
Connections:
- net 12: now also TCH5.1; no longer TCH4.1
- net 15: now also TCH3.1; no longer TCH2.1
- net 13: now reaches U1.13 (GPIO13/TCH4)
- net 13: now also TCH4.1
- net 2: now reaches U1.2 (GPIO2/TCH2)
- net 2: now also TCH2.1
- net 4: now reaches U1.4 (GPIO4/TCH0)
- net 4: now also TCH1.1
- net 0: no longer names the net of U1.0 (GPIO0/TCH1)
- net 0: no longer TCH1.1
- no-connect marks 13 -> 11
Other:
- moved on the sheet: BT1, D1, D2, D3, D4, D5, D6, D7, D8, D9, J1, R1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

Commit message: art and eda layout work
Parts:
- removed D7, D8, D9: LED_3mm, 0_local:LED_D3.0mm-2-std_back, symbol 0_local:LED_THT_3mm
- removed R7, R8, R9: 47R_6.3mm, 0_local:R_Axial_DIN0207_L6.3_D2.5_P7.62_Horiz_back, symbol 0_local:R_Axial_Z_L6.3
Connections:
- net 18: no longer names the net of U1.18 (GPIO18)
- net 23: no longer names the net of U1.23 (GPIO23)
- net 5: no longer names the net of U1.5 (GPIO5)
- no-connect marks 11 -> 14
Other:
- moved on the sheet: BT1, C10, C11, C12, C20, C21, C22, D1, D10, D11, D12, D2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

Commit message: pcb layout updates
Parts:
- added J2, J3: 01x02, 0_local:Conn_Pin_Header_Male_Horiz_Back_1x02_Pitch2.54mm, symbol 0_local:Conn_01x02
Connections:
- net 14: now also D3.2 (A); no longer D1.2 (A)
- net 25: now also D6.2 (A); no longer D4.2 (A)
- net 26: now also D5.2 (A); no longer D3.2 (A)
- net 27: now also D4.2 (A); no longer D2.2 (A)
- net 32: now also D2.2 (A); no longer D6.2 (A)
- net 33: now also D1.2 (A); no longer D5.2 (A)
- net GND: now also J2.1 (Pin_1), J2.2 (Pin_2), J3.1 (Pin_1), J3.2 (Pin_2)
Other:
- note added: "Mechanical Battery Holder"
- note added: "Two 1x2 right angle header pins and a rubber band between them hold the Lipo Battery in place"
- moved on the sheet: BT1, J1, SW1
